File: hw/sch_pcb/ADSBAFE01.kicad_pcb (KiCad board)
At the start: 2 copper layers, 50.3 x 50.3 mm, 54 parts, among them J1 MCX 6GHz 50R, J2 3.3-5V, M1 HOLE, M2 HOLE, M3 HOLE, M4 HOLE, M5 RFShield_TwoPieces, SW1 SN74LVC1G3157, SW2 SN74LVC1G3157, U1 BGA2818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

Commit message: schematic first iteration
Parts:
- removed FID1, FID2: Fiducial, Fiducial:Fiducial_1mm_Mask2mm
- added D4: SMP1330-005LF, Package_TO_SOT_SMD:SOT-23_Handsoldering, B.Cu at (122.7, 59.7)
- added J3: MCX 6GHz 50R, Mlab_CON:MCX, F.Cu at (159.0, 115.5)
- added R10: 20R, Resistor_SMD:R_0603_1608Metric_Pad0.98x0.95mm_HandSolder, B.Cu at (111.7, 105.5)
- added R11: 20R, Resistor_SMD:R_0603_1608Metric_Pad0.98x0.95mm_HandSolder, B.Cu at (111.7, 103.0)
- added R12: 20R, Resistor_SMD:R_0603_1608Metric_Pad0.98x0.95mm_HandSolder, B.Cu at (111.7, 100.4)
- added R13: 20R, Resistor_SMD:R_0603_1608Metric_Pad0.98x0.95mm_HandSolder, B.Cu at (111.7, 97.9)
- added R14: 20R, Resistor_SMD:R_0603_1608Metric_Pad0.98x0.95mm_HandSolder, B.Cu at (111.7, 95.4)
- added R15: 20R, Resistor_SMD:R_0603_1608Metric_Pad0.98x0.95mm_HandSolder, B.Cu at (111.7, 92.9)
- added R16: 20R, Resistor_SMD:R_0603_1608Metric_Pad0.98x0.95mm_HandSolder, B.Cu at (116.0, 105.5)
- added R17: 20R, Resistor_SMD:R_0603_1608Metric_Pad0.98x0.95mm_HandSolder, B.Cu at (116.0, 103.0)
- added R18: 20R, Resistor_SMD:R_0603_1608Metric_Pad0.98x0.95mm_HandSolder, B.Cu at (116.0, 100.4)
- added R19: 1k, Resistor_SMD:R_0603_1608Metric_Pad0.98x0.95mm_HandSolder, B.Cu at (116.0, 97.9)
- added R20: 1k, Resistor_SMD:R_0603_1608Metric_Pad0.98x0.95mm_HandSolder, B.Cu at (116.0, 95.4)
- added R9: 0R, Resistor_SMD:R_0603_1608Metric_Pad0.98x0.95mm_HandSolder, B.Cu at (161.0, 60.5)
- C1, C10, C11, C12, C13, C14, C15, C2, C3, C4, C5, C6, C7, C8, C9: footprint Capacitor_SMD:C_0402_1005Metric -> Capacitor_SMD:C_0603_1608Metric_Pad1.08x0.95mm_HandSolder; moved to B.Cu
- C16, C17: footprint Capacitor_SMD:C_0805_2012Metric -> Capacitor_SMD:C_0805_2012Metric_Pad1.18x1.45mm_HandSolder
- D1, D2, L1, SW1, SW2, U1, U2, U4, U5: moved to B.Cu
- J1: value MCX 6GHz 50R -> HEADER_2x02_PARALLEL; footprint Mlab_CON:MCX -> Mlab_Pin_Headers:Straight_2x02
- J2: value 3.3-5V -> HEADER_2x12_PARALLEL; footprint Mlab_Pin_Headers:Straight_2x03 -> Mlab_Pin_Headers:Straight_2x12
- R1, R2, R3, R4, R5, R6, R7, R8: footprint Resistor_SMD:R_0402_1005Metric -> Resistor_SMD:R_0603_1608Metric_Pad0.98x0.95mm_HandSolder; moved to B.Cu
- TP1, TP2, TP3, TP4, TP5, TP6, TP7, TP8: moved to F.Cu
- U3: footprint Package_SO:VSSOP-8_3.0x3.0mm_P0.65mm -> Package_SO:VSSOP-8_3x3mm_P0.65mm; moved to B.Cu
- X1: footprint Custom_Filter:Filter_SAW-6_3.8x3.8mm -> ADSB_project_footprints:Filter_SAW-6_3.8x3.8mm; moved to B.Cu
- moved J1 118.0 mm to (148.1, 126.1)
- moved U1 93.6 mm to (163.4, 60.5), turned to -90 degrees
- moved X1 93.0 mm to (161.0, 66.5), turned to 90 degrees
- moved TP1 89.7 mm to (140.6, 73.0)
- moved D1 89.0 mm to (154.1, 72.2), turned to -90 degrees
- moved TP4 88.1 mm to (140.6, 70.9)
- moved C11 86.9 mm to (147.3, 69.2), turned to -90 degrees
- moved R4 86.9 mm to (148.3, 69.2), turned to -90 degrees
- moved C1 86.9 mm to (145.3, 69.2), turned to -90 degrees
- moved R1 86.9 mm to (146.3, 69.2), turned to -90 degrees
- moved C7 86.5 mm to (153.5, 68.6)
- moved R8 86.5 mm to (143.1, 68.6)
- moved C14 85.6 mm to (142.7, 67.1), turned to 90 degrees
- moved TP8 85.4 mm to (140.5, 66.7)
- moved SW1 85.3 mm to (147.7, 66.5), turned to 90 degrees
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Connections:
- net Net-(C9-Pad1) renamed /RF_LNA_OUT
- C16 pad 1: VCC -> +3V3
- C17 pad 1: VCC -> +3V3
- D3 pad 1: VCC -> +3V3
- J1 pad 1: /RF_IN -> +3V3
- J1 pad 2: GND -> +3V3
- J2 pad 1: GND -> Net-(J2-Pad1)
- J2 pad 2: GND -> Net-(J2-Pad1)
- J2 pad 3: VCC -> Net-(J2-Pad3)
- J2 pad 4: VCC -> Net-(J2-Pad3)
Routing:
- net /RSSI_HOLD: track 5.86 -> 0.00 mm, vias 1 -> 0
- net /I2C1_SCL: track 10.1 -> 15.9 mm, vias 1 -> 2
- net +3V3: vias 8 -> 10
- net Net-(C4-Pad1): vias 0 -> 1
- net GND: vias 42 -> 37
- net /MTL_LO_PWM: vias 0 -> 1
- net /MTL_HI_PWM: vias 0 -> 1
