File: hw/sch_pcb/ADSBAFE01.kicad_sch (KiCad schematic)
At the start: 54 parts, among them J1 MCX 6GHz 50R, J2 3.3-5V, M1 HOLE, M2 HOLE, M3 HOLE, M4 HOLE, M5 RFShield_TwoPieces, SW1 SN74LVC1G3157, SW2 SN74LVC1G3157, U1 BGA2818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

Commit message: schematic first iteration
Parts:
- removed FID1, FID2: Fiducial, Fiducial:Fiducial_1mm_Mask2mm, symbol Mechanical:Fiducial
- removed J2: 3.3-5V, Mlab_Pin_Headers:Straight_2x03, symbol MLAB_HEADER:HEADER_2x03_PARALLEL
- added D4: SMP1330-005LF, Package_TO_SOT_SMD:SOT-23_Handsoldering, symbol Device:D_Dual_Series_ACK_Parallel
- added J1: HEADER_2x02_PARALLEL, Mlab_Pin_Headers:Straight_2x02, symbol MLAB_HEADER:HEADER_2x02_PARALLEL
- added J2: HEADER_2x12_PARALLEL, Mlab_Pin_Headers:Straight_2x12, symbol MLAB_HEADER:HEADER_2x12_PARALLEL
- added R10, R11, R12, R13, R14, R15, R16, R17, R18: 20R, Resistor_SMD:R_0603_1608Metric_Pad0.98x0.95mm_HandSolder, symbol Device:R
- added R19, R20: 1k, Resistor_SMD:R_0603_1608Metric_Pad0.98x0.95mm_HandSolder, symbol Device:R
- added R9: 0R, Resistor_SMD:R_0603_1608Metric_Pad0.98x0.95mm_HandSolder, symbol Device:R
- C1, C10, C11, C12, C13, C14, C15, C2, C3, C4, C5, C6, C7, C8, C9: footprint Capacitor_SMD:C_0402_1005Metric -> Capacitor_SMD:C_0603_1608Metric_Pad1.08x0.95mm_HandSolder
- C16, C17: footprint Capacitor_SMD:C_0805_2012Metric -> Capacitor_SMD:C_0805_2012Metric_Pad1.18x1.45mm_HandSolder
- R1, R2, R3, R4, R5, R6, R7, R8: footprint Resistor_SMD:R_0402_1005Metric -> Resistor_SMD:R_0603_1608Metric_Pad0.98x0.95mm_HandSolder; symbol Device:R_US -> Device:R
- SW1, SW2: symbol Custom_Analog_Switch:SN74LVC1G3157 -> ADSB_projectlib:SN74LVC1G3157
- U3: footprint Package_SO:VSSOP-8_3.0x3.0mm_P0.65mm -> Package_SO:VSSOP-8_3x3mm_P0.65mm; symbol Custom_Amplifier_Operational:TLV3542 -> ADSB_projectlib:TLV3542
- X1: footprint Custom_Filter:Filter_SAW-6_3.8x3.8mm -> ADSB_project_footprints:Filter_SAW-6_3.8x3.8mm; symbol Custom_RF_Filter:SAW-6 Filter -> ADSB_projectlib:SAW-6_Filter
- renumbered J1 to J3
Connections:
- net VCC is gone; now on net +3V3: C16.1, C17.1, D3.1 (K)
- net +3V3: now also J1.1, J1.2, R19.1, R20.1
- net DECODE: now also R13.1
- net GND: now also D4.2 (common), J1.3, J1.4, J2.11, J2.12, J2.17, J2.18, J2.5, J2.6
- net I2C1_SCL: now also R10.1, R19.2
- net I2C1_SDA: now also R11.1, R20.2
- net MTL_HI_BIAS: now also R17.1
- net MTL_HI_PWM: now also R15.1
- net MTL_LO_BIAS: now also R16.1
- net MTL_LO_PWM: now also R14.1
- net PULSES: now also R12.1
- net RF_LNA_IN: now also R9.1
- net RF_SAW_IN: now also D4.1 (A), D4.3 (K)
- net RSSI_HOLD: now also R18.1
- net RF_LNA_OUT: now reaches C9.1, U1.3
- net RF_LNA_OUT: now also R9.2
- new net: J2.10, J2.9, R13.2
- new net: J2.23, J2.24, R18.2
- new net: J2.7, J2.8, R12.2
- new net: J2.1, J2.2, R10.2
- new net: J2.15, J2.16, R15.2
- new net: J2.19, J2.20, R16.2
- new net: J2.21, J2.22, R17.2
- new net: J2.13, J2.14, R14.2
- new net: J2.3, J2.4, R11.2
Other:
- note added: "IO pin header"
- note added: "Limiter"
- note added: "bypass res or solderjumper?"
- note added: "current limiting resistors as simple IO protection, might be DNP"
- note added: "external pull-ups, might be DNP"
- note added: "limits to 10-16dBm"
- moved on the sheet: C1, C10, C11, C12, C13, C14, C15, C16, C17, C2, C3, C4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
